File: hardware/mcu-controller/mcu_controller.kicad_sch (KiCad schematic)
At the start: 49 parts, among them J1 IEC C14 inlet (L, N, PE), J2 to duplex outlet: LIGHT hot, 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, J3 hand-wheel Hall sensor, J4 knee lever sensor (pot or Hal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, J5 travel pedal (pot or Hall), J6 pressure pedal (FSR), K1 G5LE-1A 5V (motor enable), Q1 BTA08-600BW, Q2 2N7002, SW1 needle stop up/down (toggle), SW2 single stitch (push), U2 H11AA1, U3 MOC3023, U4 DRV5023 (at the hand wheel)

Commit message: MCU controller concept: wired schematic, and its write-up in the paper
The schematic is redrawn with wires: the isolation barrier runs across
the sheet, the line side above it with L and N rails, the four parts
that span it (MOC3023, relay, H11AA1, 5 V module) on it, and the control
side below, with the Nucleo's signals wired to their blocks. Power rails
use ports. The generator now places and wires parts, splits wires and
adds junctions; tools/check_mcu_netlist.py confirms KiCad's netlist
matches the intended one. Pins re-assigned for a clean layout (RELAY D4,
ZC D5, NEEDLE D11).

The motor-control paper's section 11 gains 'A first concept circuit',
with the disclaimer that it is a concept only, the circuit, pin use,
firmware outline and cautions, and the schematic as a figure.

Co-Authored-By: Claude Opus 5.5 <noreply@anthropic.com>
Claude-Session: https://claude.ai/code/session_01D8rC2JDyb9T3n3ujD2pgX4
Parts:
- removed J1: IEC C14 inlet (L, N, PE), symbol VSM:Conn_3
- removed J2: to duplex outlet: LIGHT hot, MOTOR hot, N, PE, symbol VSM:Conn_4
- removed J3: hand-wheel Hall sensor, symbol VSM:Conn_3
- removed J4: knee lever sensor (pot or Hall), symbol VSM:Conn_3
- removed J5: travel pedal (pot or Hall), symbol VSM:Conn_3
- removed J6: pressure pedal (FSR), symbol VSM:Conn_2
- removed K1: G5LE-1A 5V (motor enable), symbol VSM:Relay_SPST
- removed PS1: IRM-05-5 (5V 1A, isolated), symbol VSM:ACDC_5V
- removed Q1: BTA08-600BW, symbol VSM:Triac
- removed U2: H11AA1, symbol VSM:H11AA1
- removed U3: MOC3023, symbol VSM:MOC3023
- added J1: IEC inlet, symbol VSM:ConnR_3
- added J2: duplex outlet: PE, LIGHT, N, MOTOR, symbol VSM:ConnR_4
- added J4: knee lever, symbol VSM:ConnR_3
- added J5: travel pedal, symbol VSM:ConnR_3
- added J6: pressure pedal (FSR), symbol VSM:ConnR_2
- added K1: G5LE-1A 5V, symbol VSM:Relay_H
- added PS1: IRM-05-5, symbol VSM:ACDC_5V_H
- added Q1: BTA08-600BW, symbol VSM:Triac_R
- added U2: H11AA1, symbol VSM:H11AA1_H
- added U3: MOC3023, symbol VSM:MOC3023_H
- C2: value 47n X2 (DNP) -> 47n X2 DNP
- C5: value 100n (at sensor) -> 100n at sensor
- R6: value 100 1W (DNP) -> 100 1W DNP
- RV1: value 150VAC 14mm -> 150VAC
- RV2: value 10k lin (speed limit, panel) -> 10k speed limit
- SW1: value needle stop up/down (toggle) -> needle up/down
- SW2: value single stitch (push) -> single stitch
- U4: value DRV5023 (at the hand wheel) -> DRV5023 at hand wheel
Connections:
- net FSR_F is gone; now on net FSR: A1.CN3_10 (A2/PA3), C8.1, R19.2
- net KNEE_F is gone; now on net KNEE: A1.CN3_12 (A0/PA0), C6.1, R16.2
- net LIMIT_F is gone; now on net LIMIT: A1.CN3_9 (A3/PA4), C9.1, R20.2
- net OPTO_A is gone; now on net FIRE: R11.2
- net PEDAL_F is gone; now on net PEDAL: A1.CN3_11 (A1/PA1), C7.1, R17.2
- net ZC_B is gone; now on net N: R8.1
- net +3V3: now also J4.1, J5.1, J6.1
- net +5V: now also K1.1 (COIL+), PS1.3 (+Vo)
- net FIRE: no longer R11.1
- net FSR: no longer R18.1, R19.1
- net GATE: now also R5.2, Q1.3 (G), U3.4 (MT); no longer R5.1
- net GND: now also J4.3, J5.3, PS1.4 (-Vo), U2.4 (E), U3.2 (K)
- net HALL: now also A1.CN4_9 (D6/PB6), C4.1; no longer R14.2, U4.2 (OUT)
- net KNEE: no longer R16.1
- net LIMIT: no longer R20.1, RV2.2 (W)
- net N: now also J1.2, J2.3, PS1.2 (N); no longer R8.2
- net NEEDLE: now also A1.CN4_14 (D11/PB5); no longer A1.CN4_7 (D4/PB7)
- net PE: now also J1.3, J2.1
- net PEDAL: no longer R17.1
- net RELAY: now also A1.CN4_7 (D4/PB7); no longer A1.CN4_14 (D11/PB5)
- net ZC: now also A1.CN4_8 (D5/PA15), U2.5 (C); no longer A1.CN4_5 (D2/PA12)
- removed net HALL_F: A1.CN4_9 (D6/PB6), C4.1, R15.2
- net L_F renamed L (fused)
- net L (fused): now also J2.2, K1.3 (COM)
- net L_IN: no longer names the net of F1.1
- net L_IN: now also J1.1
- net L_K renamed MOTOR
- net MOTOR: now also R4.1, J2.4, Q1.2 (MT2); no longer R5.2
- net L_PS: no longer names the net of F2.2
- net L_PS: now also PS1.1 (L)
- net MOT_OUT renamed MT1 (via K1)
- net MT1 (via K1): now also R5.1, K1.4 (NO), Q1.1 (MT1); no longer R4.1
- net OPTO_MT: no longer names the net of R4.2
- net OPTO_MT: now also U3.6 (MT)
- net RLY_D: no longer names the net of D1.2 (A), Q2.3 (D)
- net RLY_D: now also K1.2 (COIL-)
- net RLY_G: no longer names the net of Q2.1 (G), R12.2, R13.1
- net SNUB: no longer names the net of C2.1, R6.2
- net ZC_A: no longer names the net of R7.2
- net ZC_A: now also U2.1 (AC)
- new net: R11.1, U3.1 (A)
- new net: R8.2, U2.2 (AC)
- new net: R20.1, RV2.2 (W)
- new net: J5.2, R17.1
- new net: R14.2, R15.2, U4.2 (OUT)
- new net: J4.2, R16.1
- new net: J6.2, R18.1, R19.1
Other:
- note added: "1. After Freescale AN1662: zero-cross interrupt starts a timer; at the firing delay a ~100 us gate pulse fires the triac; hand-wheel period by"
- note added: "10k speed limit"
- note added: "150VAC"
- note added: "1W DNP"
- note added: "2. Pins: FIRE D3/PB0 (TIM3_CH3 one-pulse); RELAY D4/PB7 (SB2 off); ZC D5/PA15 (SB3 off, EXTI); HALL D6/PB6 (TIM4_CH1 capture);"
- note added: "3. PS1 feeds CN3-4 (+5V): the ST-LINK is then unpowered (UM2397). Program and debug over USB with the mains unplugged, or via a USB isolator."
- note added: "4. Fire only after a zero-cross has been seen and the command is zero; close K1 last and open it first. Never scope the line side."
- note added: "47n"
- note added: "5. R7/R8: ~3.9 mA peak in the H11AA1; R11: ~8 mA into U3 from 3.3 V; R6/C2 fitted only if a snubberless triac false-fires."
- note added: "DRV5023 at hand wheel"
- note added: "G5LE-1A 5V"
- note added: "HAND-WHEEL HALL SENSOR (3-wire cable; one magnet, one pulse per stitch)"
- note added: "IEC inlet"
- note added: "IRM-05-5"
- note added: "ISOLATED 5 V"
- note added: "ISOLATION BARRIER: U3, K1, U2 and PS1 straddle it; keep at least 6 mm creepage across it"
- note added: "MAINS IN, FUSE, SURGE; OUTLET (LIGHT always on, MOTOR controlled)"
- note added: "MOTOR-ENABLE RELAY"
- note added: "NOTES. A concept drawn by Claude at Bob Drzyzgula's direction, October 2026: not built, not tested, values not checked."
- note added: "OPERATOR INPUTS (RC-filtered ADC)"
- note added: "STITCH D9/PA8; NEEDLE D11/PB5; A0-A3 knee, pedal, FSR, limit. D0/D1 left for the ST-LINK COM port. Check against the datasheet."
- note added: "SWITCHES (internal pull-ups)"
- note added: "TRIAC FIRING"
- note added: "TRIAC STAGE (after AN1662: triac in series with the motor)"
- note added: "X2 DNP"
- note added: "ZERO-CROSS"
- note added: "at sensor"
- note added: "duplex outlet: PE, LIGHT, N, MOTOR"
- note added: "input capture; speed loop every half-cycle (120 Hz); stall watchdog. Added: full isolation, motor-enable relay, operator inputs."
- note added: "knee lever"
- note added: "stitch"
- note added: "travel pedal"
- note added: "up/down"
- note removed: "(at sensor)"
- note removed: "1. After Freescale AN1662 (Skalka): zero-cross interrupt starts a timer; at the firing angle a short gate pulse (~100 us) fires the triac each half-cycle;"
- note removed: "100 1W (DNP)"
- note removed: "150VAC 14mm"
- note removed: "2. Pins: ZC on D2/PA12 (EXTI); FIRE on D3/PB0 (TIM3_CH3, one-pulse); HALL on D6/PB6 (TIM4_CH1 input capture); RELAY on D11/PB5;"
- note removed: "3. Power: PS1 feeds CN3-4 (+5V). Per UM2397 the ST-LINK is then unpowered: program and debug over USB with the mains unplugged."
- note removed: "4. Fire only after a zero-cross has been seen and the speed command is zero (no start on power-up); close K1 last, open it first."
- note removed: "47n X2 (DNP)"
- note removed: "5. Values to check: R7/R8 set H11AA1 LED current (~3.9 mA peak at 170 V); R11 gives ~8 mA into U3 from 3.3 V; Q1 needs a heatsink for long runs;"
- note removed: "6. Hall: DRV5023 unipolar switch (open drain) at the hand wheel on a 3-wire cable; one magnet gives one pulse per stitch and needle position."
- note removed: "A0-A3 = knee, pedal, FSR, speed limit; NEEDLE on D4/PB7 (SB2 must be OFF); STITCH on D9/PA8. D0/D1 left for the ST-LINK virtual COM port."
- note removed: "DRV5023 (at the hand wheel)"
- note removed: "For live debugging use a USB isolator. Never connect a scope ground to the line side."
- note removed: "G5LE-1A 5V (motor enable)"
- note removed: "HAND-WHEEL HALL SENSOR (one magnet: one pulse per stitch)"
- note removed: "IEC C14 inlet (L, N, PE)"
- note removed: "IRM-05-5 (5V 1A, isolated)"
- note removed: "ISOLATED 5 V SUPPLY"
- note removed: "ISOLATION BARRIER: U2, U3, K1, PS1 straddle it; keep >= 6 mm creepage"
- note removed: "J3"
- note removed: "MAINS IN, FUSING, SURGE"
- note removed: "MOTOR ENABLE RELAY (cuts the triac's line on a fault)"
- note removed: "NOTES (draft, Claude at Bob Drzyzgula's direction, October 2026; not built or tested)"
- note removed: "OPERATOR INPUTS (RC-filtered ADC; switches: internal pull-ups)"
- note removed: "OUTLET (base's duplex: LIGHT always on, MOTOR controlled)"
- note removed: "R6/C2 snubber is DNP with a snubberless (BW) triac and fitted if it false-fires; MOV 150 VAC for 120 V mains."
- note removed: "TRIAC FIRING (LED of U3)"
- note removed: "TRIAC STAGE (AN1662: triac in series with the motor)"
- note removed: "ZERO-CROSS DETECTOR (AN1662 uses a resistor to a pin; here isolated)"
- note removed: "hand-wheel Hall sensor"
- note removed: "knee lever sensor (pot or Hall)"
- note removed: "lin (speed limit, panel)"
- note removed: "stitch (push)"
- note removed: "stop up/down (toggle)"
- note removed: "tacho period measured by input capture; speed loop updated every half-cycle (120 Hz); stall watchdog. Added here: full isolation, relay, inputs."
- note removed: "to duplex outlet: LIGHT hot, MOTOR hot, N, PE"
- note removed: "travel pedal (pot or Hall)"
- title: VSM MCU phase controller (draft) -> VSM MCU phase controller (concept)

Commit message: MCU controller concept: retarget to the RP2350B
The schematic's controller block becomes a generic RP2350B core board,
drawn by GPIO number: FIRE GP4, RELAY GP5, ZC GP6, HALL GP7, STITCH GP10,
NEEDLE GP12, the four analog inputs on ADC0-3 (GP40-43), ADC4-7 spare.
5 V enters VSYS through a Schottky (D2), so USB can stay connected.
Netlist checked against KiCad's. The paper's section 11, the README and
the drawing's notes follow: Pico SDK in C with no RTOS, timer alarm or
PIO for the gate pulse, edge timestamps for the hand wheel, UF2 flashing.

Co-Authored-By: Claude Opus 5.5 <noreply@anthropic.com>
Claude-Session: https://claude.ai/code/session_01D8rC2JDyb9T3n3ujD2pgX4
Parts:
- removed A1: NUCLEO-G431KB, symbol VSM:NUCLEO-G431KB
- added A1: RP2350B core board, symbol VSM:RP2350B_CORE
- added D2: SS14 (Schottky), symbol VSM:D
Connections:
- net +3V3: now also A1.L14 (3V3(OUT))
- net +5V: now also D2.2 (A)
- net FIRE: now also A1.R6 (GP4)
- net FSR: now also A1.L10 (GP42/ADC2)
- net GND: now also A1.L2 (GND), A1.R4 (GND)
- net HALL: now also A1.R9 (GP7)
- net KNEE: now also A1.L12 (GP40/ADC0)
- net LIMIT: now also A1.L9 (GP43/ADC3)
- net NEEDLE: now also A1.R14 (GP12)
- net PEDAL: now also A1.L11 (GP41/ADC1)
- net RELAY: now also A1.R7 (GP5)
- net STITCH: now also A1.R12 (GP10)
- net ZC: now also A1.R8 (GP6)
- new net: A1.L4 (VSYS), D2.1 (K)
Other:
- note added: "(Schottky)"
- note added: "1. After Freescale AN1662: zero-cross interrupt sets a timer alarm (or a PIO program); at the firing delay a ~100 us gate pulse fires the"
- note added: "2. Pins (RP2350B): FIRE GP4; RELAY GP5; ZC GP6; HALL GP7; STITCH GP10; NEEDLE GP12; knee, pedal, FSR, limit on ADC0-3 (GP40-43),"
- note added: "3. PS1 feeds VSYS through D2, so USB may stay plugged in (the control side is SELV). Flash by UF2 (BOOTSEL) or SWD. Drive GP4 at 8-12 mA."
- note added: "ADC4-7 spare; GP0/GP1 UART0 for a debug line (or USB serial). Any GPIO will do for the digital signals; wire by GPIO number."
- note added: "D2"
- note added: "RP2350B CORE BOARD (pins by GPIO number)"
- note added: "RP2350B core board"
- note added: "SS14"
- note added: "triac; hand-wheel period from edge timestamps; speed loop every half-cycle (120 Hz); stall watchdog. Added: isolation, relay, inputs."
- note removed: "1. After Freescale AN1662: zero-cross interrupt starts a timer; at the firing delay a ~100 us gate pulse fires the triac; hand-wheel period by"
- note removed: "2. Pins: FIRE D3/PB0 (TIM3_CH3 one-pulse); RELAY D4/PB7 (SB2 off); ZC D5/PA15 (SB3 off, EXTI); HALL D6/PB6 (TIM4_CH1 capture);"
- note removed: "3. PS1 feeds CN3-4 (+5V): the ST-LINK is then unpowered (UM2397). Program and debug over USB with the mains unplugged, or via a USB isolator."
- note removed: "NUCLEO-32 (STM32G431KB)"
- note removed: "NUCLEO-G431KB"
- note removed: "STITCH D9/PA8; NEEDLE D11/PB5; A0-A3 knee, pedal, FSR, limit. D0/D1 left for the ST-LINK COM port. Check against the datasheet."
- note removed: "input capture; speed loop every half-cycle (120 Hz); stall watchdog. Added: full isolation, motor-enable relay, operator inputs."

Commit message: MCU controller: notes for the WeAct RP2350B Core board
From the board's schematic: GP0 links to an optional PSRAM's chip select,
GP23 is a button and GP25 the LED, and USB VBUS reaches the 5V rail
through a diode, so the supply module can feed the 5V pin directly and
D2 can be left out. The debug UART moves to GP8/GP9 (UART1), clear of
GP0. Drawing notes, README and paper section 11 updated.

Co-Authored-By: Claude Opus 5.5 <noreply@anthropic.com>
Claude-Session: https://claude.ai/code/session_01D8rC2JDyb9T3n3ujD2pgX4
Other:
- note added: "6. On a WeAct RP2350B Core board, feed PS1 to the 5V pin: the board has its own diode from USB VBUS, so D2 may be left out."
- note added: "ADC4-7 spare; GP8/GP9 UART1 for a debug line (or USB serial). Avoid GP0 (PSRAM select on some boards), GP23, GP25 (key, LED)."
- note removed: "ADC4-7 spare; GP0/GP1 UART0 for a debug line (or USB serial). Any GPIO will do for the digital signals; wire by GPIO number."

Commit message: MCU concept: heel tap and taught needle stops
From Danielle's reading of the paper: what a sewist asks of a pedal (full
power from the first movement, no heat at rest, stopping the needle up or
down where it is wanted, and the heel tap).

Schematic draft-4: a heel switch in either pedal (J5 and J6 now 4-pin),
filtered to GP11; an optional hand-wheel encoder, two DRV5013 latches in
quadrature over a ring of alternating magnets, on GP2/GP3 for a PIO
counter, beside the DRV5023 index. Heel and encoder lines join by net
labels; the generator now unions same-name labels, and its netlist still
matches KiCad's. Knee group moved up 2.54 mm and the notes tightened to
fit the sheet; the figure's crop extended.

README and paper: pin tables, firmware outline (taught stops, landing by
angle with a learned coast, heel tap, no hum below the start threshold),
and why one magnet is not enough. PARTS.md: encoder, magnets, heel switch,
4- and 5-pin connectors, passives.

Co-Authored-By: Claude Opus 5.5 <noreply@anthropic.com>
Claude-Session: https://claude.ai/code/session_01D8rC2JDyb9T3n3ujD2pgX4
Parts:
- removed J5: travel pedal, symbol VSM:ConnR_3
- removed J6: pressure pedal (FSR), symbol VSM:ConnR_2
- added C14: 100n, symbol VSM:C
- added C15, C16: 100n at sensor, symbol VSM:C
- added C17, C18: 1n, symbol VSM:C
- added J5: travel pedal + heel, symbol VSM:ConnR_4
- added J6: pressure pedal (FSR) + heel, symbol VSM:ConnR_4
- added R21: 1k, symbol VSM:R
- added R22, R23: 100, symbol VSM:R
- added R24, R25: 10k, symbol VSM:R
- added U5, U6: DRV5013 at hand wheel, symbol VSM:DRV5013
Connections:
- net +3V3: now also C15.1, C16.1, J5.1, J6.1, R24.1, R25.1, U5.1 (VCC), U6.1 (VCC)
- net GND: now also C14.2, C15.2, C16.2, C17.2, C18.2, J5.3, J6.4, U5.3 (GND), U6.3 (GND)
- net at R18.1, R19.1: now also J6.2
- net HEEL_F: now reaches A1.R13 (GP11)
- net HEEL_F: now also C14.1, R21.2
- net ENC_A: now reaches A1.R3 (GP2)
- net ENC_A: now also C17.1, R22.1
- net ENC_B: now reaches A1.R5 (GP3)
- net ENC_B: now also C18.1, R23.1
- net at R17.1: now also J5.2
- new net: R23.2, R25.2, U6.2 (OUT)
- new net: R22.2, R24.2, U5.2 (OUT)
- new net HEEL: J5.4, J6.3, R21.1
- no-connect marks 20 -> 17
Other:
- note added: "2. Pins (RP2350B): FIRE GP4; RELAY GP5; ZC GP6; HALL (index) GP7; ENC_A/B GP2/GP3 (PIO counter); STITCH GP10; HEEL GP11; NEEDLE GP12;"
- note added: "7. Heel: momentary switch to GND in either pedal (J5 pin 4, J6 pin 3); a heel tap sends the needle to its other stop."
- note added: "8. Encoder U5/U6 (ring of alternating magnets) optional: stops taught and landed by angle; 5-wire cable (3V3, GND, index, A, B)."
- note added: "C14"
- note added: "C15"
- note added: "C16"
- note added: "C17"
- note added: "C18"
- note added: "DRV5013 at hand wheel"
- note added: "HAND-WHEEL ENCODER (two Hall latches, quadrature; same cable as the index)"
- note added: "HAND-WHEEL INDEX SENSOR (one magnet, one pulse per stitch)"
- note added: "HEEL SWITCH"
- note added: "R21"
- note added: "R22"
- note added: "R23"
- note added: "R24"
- note added: "R25"
- note added: "U5"
- note added: "U6"
- note added: "knee, pedal, FSR, limit on ADC0-3 (GP40-43); ADC4-7 spare; GP8/GP9 UART1 for debug (or USB serial). Avoid GP0, GP23, GP25 (PSRAM, key, LED)."
- note added: "pressure pedal (FSR) + heel"
- note added: "travel pedal + heel"
- note removed: "2. Pins (RP2350B): FIRE GP4; RELAY GP5; ZC GP6; HALL GP7; STITCH GP10; NEEDLE GP12; knee, pedal, FSR, limit on ADC0-3 (GP40-43),"
- note removed: "ADC4-7 spare; GP8/GP9 UART1 for a debug line (or USB serial). Avoid GP0 (PSRAM select on some boards), GP23, GP25 (key, LED)."
- note removed: "HAND-WHEEL HALL SENSOR (3-wire cable; one magnet, one pulse per stitch)"
- note removed: "pressure pedal (FSR)"
- note removed: "travel pedal"

Commit message: MCU concept: optional motor-current transformer (T1)
A ZMCT103C-class 1000:1 current transformer straddling the barrier, the
motor's hot lead through its window, for sensorless IR compensation. On
the control side: a 100 ohm burden (about 0.1 V per amp), a 1.65 V bias
from a 10k/10k divider with 10 uF, and a 1k/10n filter into ADC4 (GP44),
joined by the ISENSE label. Netlist still matches KiCad's. README, paper
(barrier parts, pin table, load-compensation note) and parts list
updated.

Co-Authored-By: Claude Opus 5.5 <noreply@anthropic.com>
Claude-Session: https://claude.ai/code/session_01D8rC2JDyb9T3n3ujD2pgX4
Parts:
- added C19: 10n, symbol VSM:C
- added C20: 10u, symbol VSM:C
- added R26: 100 burden, symbol VSM:R
- added R27: 1k, symbol VSM:R
- added R28, R29: 10k, symbol VSM:R
- added T1: ZMCT103C 1000:1 (optional), symbol VSM:CT_H
Connections:
- net +3V3: now also R28.1
- net GND: now also C19.2, C20.2, R29.2
- net MOTOR: now also T1.1 (P); no longer C2.2, Q1.2 (MT2), R4.1
- net ISENSE: now reaches A1.L8 (GP44/ADC4)
- net ISENSE: now also C19.1, R27.2
- new net: C2.2, Q1.2 (MT2), R4.1, T1.2 (P)
- new net: C20.1, R26.2, R28.2, R29.1, T1.3 (S1)
- new net: R26.1, R27.1, T1.4 (S2)
- no-connect marks 17 -> 16
Other:
- note added: "10n"
- note added: "5. R7/R8: ~3.9 mA peak in the H11AA1; R11: ~8 mA into U3 from 3.3 V; R6/C2 fitted only if a snubberless triac false-fires. T1 optional: motor lead through its window, 0.1 V/A about 1.65 V."
- note added: "C19"
- note added: "C20"
- note added: "ISOLATION BARRIER: U3, K1, U2, PS1 (and T1) straddle it; keep at least 6 mm creepage across it"
- note added: "MOTOR CURRENT (optional)"
- note added: "R26"
- note added: "R27"
- note added: "R28"
- note added: "R29"
- note added: "T1"
- note added: "ZMCT103C 1000:1 (optional)"
- note added: "burden"
- note added: "knee, pedal, FSR, limit on ADC0-3 (GP40-43); ISENSE ADC4; ADC5-7 spare; GP8/GP9 UART1 for debug (or USB serial). Avoid GP0, GP23, GP25 (PSRAM, key, LED)."
- note removed: "5. R7/R8: ~3.9 mA peak in the H11AA1; R11: ~8 mA into U3 from 3.3 V; R6/C2 fitted only if a snubberless triac false-fires."
- note removed: "ISOLATION BARRIER: U3, K1, U2 and PS1 straddle it; keep at least 6 mm creepage across it"
- note removed: "knee, pedal, FSR, limit on ADC0-3 (GP40-43); ADC4-7 spare; GP8/GP9 UART1 for debug (or USB serial). Avoid GP0, GP23, GP25 (PSRAM, key, LED)."
